File: calculator2.sch (EAGLE design)
At the start: 41 parts

Commit message: Using 32 board
Parts:
- removed DISPLAY: (no value), adafruit:PINHD-1X9
- removed G1: CR2032H, battery:CR2032H
- removed U$1: TEENSY41, teensy:TEENSY41
- added CHARGER: PROTRINKET, pwlib:PROTRINKET
- added CONTROLLER: IB32U4, pwlib:IB32U4
- added LIPO: (no value), pinhead:PINHD-1X2
- added SHARPMEM: SHARPMEM, pwlib:SHARPMEM
Connections:
- removed net N$2: G1.+, U$1.VBAT
- removed net SCK: DISPLAY.4, U$1.13-SCK/LED
- new net N$1: CHARGER.BAT, CONTROLLER.BATT, LIPO.1
- new net SLCK: CONTROLLER.SCK, SHARPMEM.SLCK
- new net VHI: CHARGER.+5V, CONTROLLER.VHI
- net 3V3: now also CONTROLLER.3V3, SHARPMEM.VIN; no longer DISPLAY.1, U$1.3V3-1, U$1.3V3-2
- net C1: now also CONTROLLER.7; no longer U$1.9-OUT1C
- net C2: now also CONTROLLER.1; no longer U$1.8-TX2/IN1
- net C3: now also CONTROLLER.0; no longer U$1.7-RX2/OUT1A
- net C4: now also CONTROLLER.4; no longer U$1.6-OUT1D
- net C5: now also CONTROLLER.A2; no longer U$1.1-TX1/MISO1/CTX2
- net CL: now also CONTROLLER.12; no longer U$1.27-A13/SCK1
- net CS: now also CONTROLLER.A5, SHARPMEM.CS; no longer DISPLAY.6, U$1.10-CS/MQSR
- net EX: now also CONTROLLER.A3; no longer U$1.0-RX1/CS1/CRX2
- net GND: now also CHARGER.GND, LIPO.2, SHARPMEM.GND; no longer DISPLAY.3, G1.-, U$1.GND1, U$1.GND2, U$1.GND3
- net MOSI: now also CONTROLLER.MOSI, SHARPMEM.MOSI; no longer DISPLAY.5, U$1.11-MOSI/CTX1
- net R1: now also CONTROLLER.A1; no longer U$1.2-OUT2
- net R2: now also CONTROLLER.6; no longer U$1.5-IN2
- net R3: now also CONTROLLER.8; no longer U$1.4-BCLK2
- net R4: now also CONTROLLER.A0; no longer U$1.3-LRCLK2
- net R5: now also CONTROLLER.9; no longer U$1.24-A10/TX6/SCL2
- net R6: now also CONTROLLER.10; no longer U$1.25-A11/RX6/SDA2
- net R7: now also CONTROLLER.11; no longer U$1.26-A12/MOSI1
- net SH: now also CONTROLLER.13; no longer U$1.28-RX7
