File: calculator3.brd (EAGLE design)
At the start: 73 x 140 mm, 41 parts

Commit message: Pins confirmed
Connections:
- removed net N$1 (its old number): CONTROLLER.13
- removed net N$10: CONTROLLER.10
- removed net N$11: CONTROLLER.9
- removed net N$12: CONTROLLER.7
- removed net N$13: CONTROLLER.A1
- removed net N$14: CONTROLLER.A2
- removed net N$15: CONTROLLER.A3
- removed net N$16: CONTROLLER.A4
- removed net N$17: CONTROLLER.1
- removed net N$18: CONTROLLER.0
- removed net N$19: CONTROLLER.RST
- removed net N$2 (its old number): CONTROLLER.12
- removed net N$20: CONTROLLER.4
- removed net N$21: CONTROLLER.3
- removed net N$3: CONTROLLER.VHI
- removed net N$8: CONTROLLER.A0
- removed net N$9: CLR.3, JP2.4
- new net BAT: CHARGER.BAT, CONTROLLER.BAT
- new net VHI: CHARGER.5V, CONTROLLER.VHI
- net CLR: now also CLR.3, JP2.4
- net COL1: now also CONTROLLER.10
- net COL2: now also CONTROLLER.9
- net COL3: now also CONTROLLER.7
- net COL4: now also CONTROLLER.A1
- net COL5: now also CONTROLLER.A3
- net COL6: now also CONTROLLER.A4
- net EXIT: now also CONTROLLER.RST
- net GND: now also CHARGER.GND
- net ROW1: now also CONTROLLER.A2
- net ROW2: now also CONTROLLER.A0
- net ROW3: now also CONTROLLER.13
- net ROW4: now also CONTROLLER.1
- net ROW5: now also CONTROLLER.0
- net ROW6: now also CONTROLLER.4
- net ROW7: now also CONTROLLER.3
- net SHIFT: now also CONTROLLER.12
Routing:
- net CLR: track 14.6 -> 130.9 mm
- net N$9: track 114.5 -> 0.00 mm
- net BAT: track 0.00 -> 72.0 mm
- net VHI: track 0.00 -> 47.2 mm
- net N$3: track 45.0 -> 0.00 mm
- net ROW5: track 161.0 -> 179.4 mm
- net GND: track 352.8 -> 370.9 mm
- net ROW4: track 149.7 -> 166.2 mm
- net EXIT: track 166.6 -> 172.8 mm
- net ROW2: track 140.6 -> 146.2 mm
- net COL4: track 152.2 -> 157.6 mm
- net ROW3: track 141.8 -> 147.2 mm
- net ROW1: track 139.5 -> 144.7 mm
- net COL6: track 158.3 -> 163.3 mm
- net COL5: track 98.8 -> 103.8 mm
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- added copper zone on layer 16, net GND
Other:
- board text added: "R3 SH R2 CLR C1 C2 C3 C4 R1 C5 C6 R4 R5 EX R6 R7 G"
