File: calculator3.sch (EAGLE design)
At the start: 41 parts

Commit message: Pins confirmed
Connections:
- removed net N$1 (its old number): CONTROLLER.13
- removed net N$10: CONTROLLER.10
- removed net N$11: CONTROLLER.9
- removed net N$12: CONTROLLER.7
- removed net N$13: CONTROLLER.A1
- removed net N$14: CONTROLLER.A2
- removed net N$15: CONTROLLER.A3
- removed net N$16: CONTROLLER.A4
- removed net N$17: CONTROLLER.1
- removed net N$18: CONTROLLER.0
- removed net N$19: CONTROLLER.RST
- removed net N$2 (its old number): CONTROLLER.12
- removed net N$20: CONTROLLER.4
- removed net N$21: CONTROLLER.3
- removed net N$3: CONTROLLER.VHI
- removed net N$8: CONTROLLER.A0
- removed net N$9: CLR.2, JP2.4
- new net BAT: CHARGER.BAT, CONTROLLER.BAT
- new net VHI: CHARGER.5V, CONTROLLER.VHI
- net CLR: now also CLR.2, JP2.4
- net COL1: now also CONTROLLER.10
- net COL2: now also CONTROLLER.9
- net COL3: now also CONTROLLER.7
- net COL4: now also CONTROLLER.A1
- net COL5: now also CONTROLLER.A3
- net COL6: now also CONTROLLER.A4
- net EXIT: now also CONTROLLER.RST
- net GND: now also CHARGER.GND
- net ROW1: now also CONTROLLER.A2
- net ROW2: now also CONTROLLER.A0
- net ROW3: now also CONTROLLER.13
- net ROW4: now also CONTROLLER.1
- net ROW5: now also CONTROLLER.0
- net ROW6: now also CONTROLLER.4
- net ROW7: now also CONTROLLER.3
- net SHIFT: now also CONTROLLER.12
Other:
- moved on the sheet: CHARGER, CONTROLLER, SHARPMEM
